Commit message: added platform modle

File: agents/chiny/chiny.xacro (robot description, xacro)
@@ -8,7 +8,7 @@
   <xacro:property name="namespace" value="chiny" />
   <xacro:property name="use_mesh_file" value="true" />
-  <xacro:property name="mesh_file" value="package://fcu_sim/meshes/firefly.dae" />
+  <xacro:property name="mesh_file" value="package://fcu_sim/meshes/hummingbird.dae" />
   <xacro:property name="mass" value="2.856" />
-  <xacro:property name="body_width" value="0.505" />
+  <xacro:property name="body_width" value="0.080" />
   <xacro:property name="body_height" value="0.1" />
   <xacro:property name="body_inertia">
@@ -26,8 +26,8 @@
       <geometry>
         <xacro:if value="${use_mesh_file}">
-          <mesh filename="${mesh_file}" scale="1 1 1" />
+          <mesh filename="${mesh_file}" scale=".3 .3 .3" />
         </xacro:if>
         <xacro:unless value="${use_mesh_file}">
-          <cylinder length="${body_height}" radius="${body_width}"/>
+          <cylinder length="${body_height}" radius="${body_width/2}"/>
         </xacro:unless>
       </geometry>
@@ -36,5 +36,5 @@
       <origin xyz="0 0 0" rpy="0 0 0" />
       <geometry>
-        <cylinder length="${body_height}" radius="${body_width}"/>
+        <cylinder length="${body_height}" radius="${body_width/2}"/>
       </geometry>
     </collision>

Commit message: made camera face up; deleted most waypoints and made waypoint threshold lower

File: agents/chiny/chiny.xacro (robot description, xacro)
@@ -66,5 +66,5 @@
     image_topic="rgb"
     image_camera_info_topic="camera_info">
-    <origin xyz="${body_width+0.1} 0 0" rpy="0 0 0"/>
+    <origin xyz="0 0 0" rpy="0 -1.5707 0"/>
   </xacro:simple_camera>
 </robot>

Commit message: added note about visualizing the camera.xacro

File: agents/chiny/chiny.xacro (robot description, xacro)
@@ -68,3 +68,19 @@
     <origin xyz="0 0 0" rpy="0 -1.5707 0"/>
   </xacro:simple_camera>
+  <!-- to visualize the camera's pose: -->
+  <!--     put the <visual> tag in the -->
+  <!--     camera.xacro as shown below -->
+<!--   <link name="${namespace}/camera_base_link">
+    <inertial>
+      <mass value="0.001"/>
+      <xacro:insert_block name="origin"/>
+      <xacro:insert_block name="empty_inertia"/>
+    </inertial>
+    <visual name="${namespace}/camera_visual">
+      <xacro:insert_block name="origin"/>
+      <geometry>
+        <sphere radius="0.009"/>
+      </geometry>
+    </visual>
+  </link> -->
 </robot>

Commit message: added a chinywhoop dae model and tuned collision -- removed the table because of weird gazebo friction interactions that caused (1) platform to shake/slip and (2) the table to sink into the ground a little bit

File: agents/chiny/chiny.xacro (robot description, xacro)
@@ -8,8 +8,8 @@
   <xacro:property name="namespace" value="chiny" />
   <xacro:property name="use_mesh_file" value="true" />
-  <xacro:property name="mesh_file" value="package://fcu_sim/meshes/hummingbird.dae" />
+  <xacro:property name="mesh_file" value="package://desktopquad_sim/agents/chiny/chinywhoop.dae" />
   <xacro:property name="mass" value="2.856" />
-  <xacro:property name="body_width" value="0.080" />
-  <xacro:property name="body_height" value="0.1" />
+  <xacro:property name="body_width" value="0.085" />
+  <xacro:property name="body_height" value="0.01" />
   <xacro:property name="body_inertia">
     <inertia ixx="0.07" ixy="0.0" ixz="0.0" iyy="0.08" iyz="0.0" izz="0.12" />
@@ -26,15 +26,15 @@
       <geometry>
         <xacro:if value="${use_mesh_file}">
-          <mesh filename="${mesh_file}" scale=".3 .3 .3" />
+          <mesh filename="${mesh_file}" scale="1 1 1" />
         </xacro:if>
         <xacro:unless value="${use_mesh_file}">
-          <cylinder length="${body_height}" radius="${body_width/2}"/>
+          <box size="${body_width} ${body_width} ${body_height}" />
         </xacro:unless>
       </geometry>
     </visual>
     <collision>
-      <origin xyz="0 0 0" rpy="0 0 0" />
+      <origin xyz="0 0 0.005" rpy="0 0 0" />
       <geometry>
-        <cylinder length="${body_height}" radius="${body_width/2}"/>
+        <box size="${body_width} ${body_width} ${body_height}" />
       </geometry>
     </collision>

Commit message: tf madness

File: agents/chiny/chiny.xacro (robot description, xacro)
@@ -66,5 +66,5 @@
     image_topic="rgb"
     image_camera_info_topic="camera_info">
-    <origin xyz="0 0 0" rpy="0 -1.5707 0"/>
+    <origin xyz="0 0 0.002" rpy="0 -1.5707 0"/>
   </xacro:simple_camera>
   <!-- to visualize the camera's pose: -->

Commit message: made camera orientation same as chiny hw

File: agents/chiny/chiny.xacro (robot description, xacro)
@@ -66,5 +66,5 @@
     image_topic="rgb"
     image_camera_info_topic="camera_info">
-    <origin xyz="0 0 0.002" rpy="0 -1.5707 0"/>
+    <origin xyz="0 0 0.002" rpy="0 -1.5707 1.5707"/>
   </xacro:simple_camera>
   <!-- to visualize the camera's pose: -->
